File: _autosave-tp4056.kicad_sch (KiCad schematic)
At the start: 26 parts, among them J1 Conn_01x01_Pin, J2 Conn_01x01_Female, J3 Conn_01x01_Female, J4 Conn_01x01_Female, J5 Conn_01x01_Female, J6 Conn_01x03_MountingPin, J7 Conn_01x01_Female, J8 USB_C_Receptacle_USB2.0, U1 TP4056, U2 DW01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

Commit message: Final Project Push
Parts:
- J1: footprint (none) -> Connector_PinHeader_2.54mm:PinHeader_1x01_P2.54mm_Vertical
Changed lines of the file:
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@@
 			)
 		)
-		(property "Footprint" ""
+		(property "Footprint" "Connector_PinHeader_2.54mm:PinHeader_1x01_P2.54mm_Vertical"
 			(at 80.01 71.12 0)
 			(effects
