File: tp4056.kicad_sch (KiCad schematic)
At the start: 26 parts, among them J1 Conn_01x01_Pin, J2 Conn_01x01_Female, J3 Conn_01x01_Female, J4 Conn_01x01_Female, J5 Conn_01x01_Female, J6 Conn_01x03_MountingPin, J7 Conn_01x01_Female, J8 USB_C_Receptacle_USB2.0, U1 TP4056, U2 DW01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

Commit message: actual changes: moved components around to free some space, added power path outputting on J1, enlarged via under the package to make soldering-iron rework possible, made PROG resistor 0805; designator placement kept reasonable
Parts:
- added D3: SS14, Diode_SMD:D_SMA, symbol Device:D_Schottky_Small
- added Q1: Q_PMOS_GSD, Package_TO_SOT_SMD:SOT-23, symbol Device:Q_PMOS_GSD
- added R11: 2k, Resistor_SMD:R_0603_1608Metric_Pad0.98x0.95mm_HandSolder, symbol Device:R_Small
- J1: footprint (none) -> Connector_PinSocket_2.54mm:PinSocket_1x01_P2.54mm_Vertical
- R3: value 10k -> 2k
Connections:
- net BAT+: now also Q1.3 (D)
- net Earth: now also R11.2
- net VIN: now also D3.2 (A), Q1.1 (G), R11.1; no longer J1.1 (Pin_1)
- new net VSYS: D3.1 (K), J1.1 (Pin_1), Q1.2 (S)
Other:
- moved on the sheet: J1
